File: Schematics/KiCad/mux side A (1-4).kicad_sch (KiCad schematic)
At the start: 150 parts, among them J1 348260240, J13 348260240, J14 348260240, J15 348260240, J16 348260240, J17 348260240, J2 348260240, J3 348260240, J4 348260240, J5 348260240, U1 CD74HC4067SM, U17 CD74HC4067SM, U18 CD74HC4067SM, U19 CD74HC4067SM, U2 CD74HC4067SM, U20 CD74HC4067SM, U3 CD74HC4067SM, U4 CD74HC4067SM, U5 CD74HC4067SM, U8 CD74HC4067SM

Commit message: Fix all errors and warnings
Parts:
- removed C22, C28, C29, C3, C30, C31, C4, C5, C6, C7: GRM033R61A104KE15D, FP-GRM033-0_03-IPC_C, symbol Altium Content Vault:mux side left_0_b4654b650e69147ec39a6b967a45e02_Altium Con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
- removed R1, R10, R11, R12, R127, R128, R129, R13, R130, R131, R132, R133, R134, R135, R136, R137, R138, R139, R14, R140, R141, R142, R143, R144, R145, R146, R147, R148, R149, R15, R150, R151, R152, R153, R154, R155, R156, R157, R158, R159, R16, R160, R161, R162, R163, R164, R165, R166, R167, R168, R169, R17, R170, R171, R172, R173, R174, R175, R176, R177, R178, R179, R18, R180, R181, R182, R183, R184, R185, R186, R19, R2, R20, R21, R22, R23, R24, R25, R26, R27, R28, R29, R3, R30, R31, R32, R33, R34, R35, R36, R37, R38, R39, R4, R40, R41, R42, R43, R44, R45, R46, R47, R48, R49, R5, R50, R51, R52, R53, R54, R55, R56, R57, R58, R59, R6, R60, R7, R8, R9: RN73R2BTTD3001B25, FP-RN73R2B-IPC_A, symbol Altium Content Vault:mux side left_0_mirrored_1029c3af85768c4190bb7ad29bc67b5_A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
- added C13, C17, C2, C22, C24, C3, C4, C5, C6, C7: 100n, Capacitor_SMD:C_0603_1608Metric, symbol Device:C
- added R1, R10, R100, R101, R102, R103, R104, R105, R106, R107, R108, R109, R11, R110, R111, R112, R113, R114, R115, R116, R117, R118, R119, R12, R120, R121, R122, R123, R124, R125, R13, R14, R15, R16, R17, R18, R19, R2, R20, R21, R22, R23, R24, R25, R26, R27, R28, R29, R3, R30, R31, R32, R33, R34, R35, R36, R37, R38, R39, R4, R40, R41, R42, R43, R44, R45, R46, R47, R48, R49, R5, R50, R51, R52, R53, R54, R55, R56, R57, R58, R59, R6, R60, R66, R67, R68, R69, R7, R70, R71, R72, R73, R74, R75, R76, R77, R78, R79, R8, R80, R81, R82, R83, R84, R85, R86, R87, R88, R89, R9, R90, R91, R92, R93, R94, R95, R96, R97, R98, R99: 3k, Resistor_SMD:R_0603_1608Metric, symbol Device:R_US
Connections:
- net +3V3: now also R1.1, R10.1, R100.1, R101.1, R102.1, R103.1, R104.1, R105.1, R106.1, R107.1, R108.1, R109.1, R11.1, R110.1, R111.1, R112.1, R113.1, R114.1, R115.1, R116.1, R117.1, R118.1, R119.1, R12.1, R120.1, R121.1, R122.1, R123.1, R124.1, R125.1, R13.1, R14.1, R15.1, R16.1, R17.1, R18.1, R19.1, R2.1, R20.1, R21.1, R22.1, R23.1, R24.1, R25.1, R26.1, R27.1, R28.1, R29.1, R3.1, R30.1, R31.1, R32.1, R33.1, R34.1, R35.1, R36.1, R37.1, R38.1, R39.1, R4.1, R40.1, R41.1, R42.1, R43.1, R44.1, R45.1, R46.1, R47.1, R48.1, R49.1, R5.1, R50.1, R51.1, R52.1, R53.1, R54.1, R55.1, R56.1, R57.1, R58.1, R59.1, R6.1, R60.1, R66.1, R67.1, R68.1, R69.1, R7.1, R70.1, R71.1, R72.1, R73.1, R74.1, R75.1, R76.1, R77.1, R78.1, R79.1, R8.1, R80.1, R81.1, R82.1, R83.1, R84.1, R85.1, R86.1, R87.1, R88.1, R89.1, R9.1, R90.1, R91.1, R92.1, R93.1, R94.1, R95.1, R96.1, R97.1, R98.1, R99.1
- net GND: now also C13.2, C17.2, C2.2, C22.2, C24.2, C3.2, C4.2, C5.2, C6.2, C7.2
- net MUX 0: now also C24.1
- net MUX 1: now also C22.1
- net MUX 2: now also C17.1
- net MUX 3: now also C13.1
- net MUX 4: now also C7.1
- net MUX 5: now also C2.1
- net MUX 6: now also C3.1
- net MUX 7: now also C4.1
- net MUX 8: now also C5.1
- net MUX 9: now also C6.1
- net S0: now also U1.10 (S0), U17.10 (S0), U18.10 (S0), U19.10 (S0), U2.10 (S0), U20.10 (S0), U3.10 (S0), U4.10 (S0), U5.10 (S0), U8.10 (S0)
- net S1: now also U1.11 (S1), U17.11 (S1), U18.11 (S1), U19.11 (S1), U2.11 (S1), U20.11 (S1), U3.11 (S1), U4.11 (S1), U5.11 (S1), U8.11 (S1)
- net S2: now also U1.14 (S2), U17.14 (S2), U18.14 (S2), U19.14 (S2), U2.14 (S2), U20.14 (S2), U3.14 (S2), U4.14 (S2), U5.14 (S2), U8.14 (S2)
- net S3: now also U1.13 (S3), U17.13 (S3), U18.13 (S3), U19.13 (S3), U2.13 (S3), U20.13 (S3), U3.13 (S3), U4.13 (S3), U5.13 (S3), U8.13 (S3)
- net at J17.1, U20.9 (I0): now also R114.2
- net at J17.11, U20.4 (I5): now also R119.2
- net at J17.13, U20.3 (I6): now also R120.2
- net at J17.15, U20.2 (I7): now also R121.2
- net at J17.17, U20.23 (I8): now also R122.2
- net at J17.19, U20.22 (I9): now also R123.2
- net at J17.21, U20.21 (I10): now also R124.2
- net at J17.23, U20.20 (I11): now also R125.2
- net at J17.3, U20.8 (I1): now also R115.2
- net at J17.5, U20.7 (I2): now also R116.2
- net at J17.7, U20.6 (I3): now also R117.2
- net at J17.9, U20.5 (I4): now also R118.2
- net at J1.3, U1.8 (I1): now also R23.2
- net at J2.15, U2.2 (I7): now also R29.2
- net at J2.23, U2.20 (I11): now also R25.2
- net at J2.21, U2.21 (I10): now also R26.2
- net at J2.19, U2.22 (I9): now also R27.2
- net at J2.17, U2.23 (I8): now also R28.2
- net at J2.13, U2.3 (I6): now also R30.2
- net at J2.11, U2.4 (I5): now also R31.2
- net at J2.9, U2.5 (I4): now also R32.2
- net at J2.7, U2.6 (I3): now also R33.2
- net at J2.5, U2.7 (I2): now also R34.2
- net at J2.3, U2.8 (I1): now also R35.2
- net at J2.1, U2.9 (I0): now also R36.2
- net at J15.11, U18.4 (I5): now also R95.2
- net at J13.5, U8.7 (I2): now also R10.2
- net at J4.23, U4.20 (I11): now also R49.2
- net at J1.19, U1.22 (I9): now also R15.2
- net at J15.15, U18.2 (I7): now also R97.2
- net at J15.23, U18.20 (I11): now also R101.2
- net at J15.21, U18.21 (I10): now also R100.2
- net at J15.19, U18.22 (I9): now also R99.2
- net at J15.17, U18.23 (I8): now also R98.2
- net at J15.13, U18.3 (I6): now also R96.2
- net at J15.9, U18.5 (I4): now also R94.2
- net at J15.7, U18.6 (I3): now also R93.2
- net at J15.5, U18.7 (I2): now also R92.2
- net at J15.3, U18.8 (I1): now also R91.2
- net at J15.1, U18.9 (I0): now also R90.2
- net at J14.11, U17.4 (I5): now also R83.2
- net at J3.1, U3.9 (I0): now also R48.2
- net at J3.11, U3.4 (I5): now also R43.2
- net at J3.13, U3.3 (I6): now also R42.2
- net at J3.15, U3.2 (I7): now also R41.2
- net at J3.17, U3.23 (I8): now also R40.2
- net at J3.19, U3.22 (I9): now also R39.2
- net at J3.21, U3.21 (I10): now also R38.2
- net at J3.23, U3.20 (I11): now also R37.2
- net at J3.3, U3.8 (I1): now also R47.2
- net at J3.5, U3.7 (I2): now also R46.2
- net at J3.7, U3.6 (I3): now also R45.2
- net at J3.9, U3.5 (I4): now also R44.2
- net at J4.15, U4.2 (I7): now also R53.2
- net at J4.21, U4.21 (I10): now also R50.2
- net at J4.19, U4.22 (I9): now also R51.2
- net at J4.17, U4.23 (I8): now also R52.2
- net at J4.13, U4.3 (I6): now also R54.2
- net at J4.11, U4.4 (I5): now also R55.2
- net at J4.9, U4.5 (I4): now also R56.2
- net at J4.7, U4.6 (I3): now also R57.2
- net at J4.5, U4.7 (I2): now also R58.2
- net at J4.3, U4.8 (I1): now also R59.2
- net at J4.1, U4.9 (I0): now also R60.2
- net at J13.9, U8.5 (I4): now also R8.2
- net at J1.13, U1.3 (I6): now also R18.2
- net at J16.3, U19.8 (I1): now also R103.2
- net at J13.7, U8.6 (I3): now also R9.2
- net at J1.15, U1.2 (I7): now also R17.2
- net at J1.23, U1.20 (I11): now also R13.2
- net at J1.21, U1.21 (I10): now also R14.2
- net at J1.17, U1.23 (I8): now also R16.2
- net at J1.11, U1.4 (I5): now also R19.2
- net at J1.9, U1.5 (I4): now also R20.2
- net at J1.7, U1.6 (I3): now also R21.2
- net at J1.5, U1.7 (I2): now also R22.2
- net at J1.1, U1.9 (I0): now also R24.2
- net at J13.11, U8.4 (I5): now also R7.2
- net at J14.5, U17.7 (I2): now also R80.2
- net at J5.1, U5.9 (I0): now also R77.2
- net at J5.3, U5.8 (I1): now also R76.2
- net at J16.9, U19.5 (I4): now also R106.2
- net at J5.15, U5.2 (I7): now also R70.2
- net at J14.15, U17.2 (I7): now also R85.2
- net at J14.23, U17.20 (I11): now also R89.2
- net at J16.11, U19.4 (I5): now also R107.2
- net at J16.15, U19.2 (I7): now also R109.2
- net at J14.1, U17.9 (I0): now also R78.2
- net at J14.13, U17.3 (I6): now also R84.2
- net at J14.17, U17.23 (I8): now also R86.2
- net at J14.19, U17.22 (I9): now also R87.2
- net at J14.21, U17.21 (I10): now also R88.2
- net at J14.3, U17.8 (I1): now also R79.2
- net at J14.7, U17.6 (I3): now also R81.2
- net at J14.9, U17.5 (I4): now also R82.2
- net at J5.11, U5.4 (I5): now also R72.2
- net at J16.23, U19.20 (I11): now also R113.2
- net at J16.21, U19.21 (I10): now also R112.2
- net at J16.19, U19.22 (I9): now also R111.2
- net at J16.17, U19.23 (I8): now also R110.2
- net at J16.13, U19.3 (I6): now also R108.2
- net at J16.7, U19.6 (I3): now also R105.2
- net at J16.5, U19.7 (I2): now also R104.2
- net at J16.1, U19.9 (I0): now also R102.2
- net at J13.19, U8.22 (I9): now also R3.2
- net at J5.23, U5.20 (I11): now also R66.2
- net at J5.13, U5.3 (I6): now also R71.2
- net at J13.3, U8.8 (I1): now also R11.2
- net at J13.1, U8.9 (I0): now also R12.2
- net at J13.13, U8.3 (I6): now also R6.2
- net at J13.15, U8.2 (I7): now also R5.2
- net at J13.17, U8.23 (I8): now also R4.2
- net at J13.21, U8.21 (I10): now also R2.2
- net at J13.23, U8.20 (I11): now also R1.2
- net at J5.9, U5.5 (I4): now also R73.2
- net at J5.21, U5.21 (I10): now also R67.2
- net at J5.19, U5.22 (I9): now also R68.2
- net at J5.17, U5.23 (I8): now also R69.2
- net at J5.7, U5.6 (I3): now also R74.2
- net at J5.5, U5.7 (I2): now also R75.2

Commit message: Condense layout to 2 layers
Parts:
- removed J14, J15, J16, J17: 348260240, TempSenseFootprints:CONN_SD-34826-001_24_MOL, symbol TempSenseSymbols:348260240
- added J10, J11, J6, J9: 348260240, CONN_SD-34826-001_24_MOL, symbol TempSenseSymbols:348260240
- J1, J13, J2, J3, J4, J5: footprint TempSenseFootprints:CONN_SD-34826-001_24_MOL -> CONN_SD-34826-001_24_MOL
Connections:
- net GND: now also J1.11, J1.13, J1.15, J1.19, J1.21, J1.23, J13.11, J13.13, J13.15, J13.19, J13.21, J13.23, J2.11, J2.13, J2.15, J2.19, J2.21, J2.23, J3.11, J3.13, J3.15, J3.19, J3.21, J3.23, J4.11, J4.13, J4.15, J4.19, J4.21, J4.23, J5.11, J5.13, J5.15, J5.19, J5.21, J5.23, J10.11, J10.12, J10.13, J10.14, J10.15, J10.16, J10.19, J10.20, J10.21, J10.22, J10.23, J10.24, J11.11, J11.12, J11.13, J11.14, J11.15, J11.16, J11.19, J11.20, J11.21, J11.22, J11.23, J11.24, J6.11, J6.12, J6.13, J6.14, J6.15, J6.16, J6.19, J6.20, J6.21, J6.22, J6.23, J6.24, J9.11, J9.12, J9.13, J9.14, J9.15, J9.16, J9.19, J9.20, J9.21, J9.22, J9.23, J9.24; no longer J1.10, J1.18, J1.2, J1.4, J1.6, J1.8, J13.10, J13.18, J13.2, J13.4, J13.6, J13.8, J2.10, J2.18, J2.2, J2.4, J2.6, J2.8, J3.10, J3.18, J3.2, J3.4, J3.6, J3.8, J4.10, J4.18, J4.2, J4.4, J4.6, J4.8, J5.10, J5.18, J5.2, J5.4, J5.6, J5.8
- net at R47.2, U3.8 (I1): now also J3.2; no longer J3.3
- net at R114.2: now also U20.20 (I11), J11.18; no longer U20.9 (I0)
- net at U20.4 (I5): now also R120.2, J11.6; no longer R119.2
- net at U20.3 (I6): now also R119.2, J11.7; no longer R120.2
- net at U20.2 (I7): now also R118.2, J11.8; no longer R121.2
- net at U20.23 (I8): now also R117.2, J11.9; no longer R122.2
- net at U20.22 (I9): now also R116.2, J11.10; no longer R123.2
- net at U20.21 (I10): now also R115.2, J11.17; no longer R124.2
- net at R125.2: now also U20.9 (I0), J11.1; no longer U20.20 (I11)
- net at U20.8 (I1): now also R124.2, J11.2; no longer R115.2
- net at U20.7 (I2): now also R123.2, J11.3; no longer R116.2
- net at U20.6 (I3): now also R122.2, J11.4; no longer R117.2
- net at U20.5 (I4): now also R121.2, J11.5; no longer R118.2
- net at R29.2, U2.2 (I7): now also J2.8; no longer J2.15
- net at R25.2, U2.20 (I11): now also J2.18; no longer J2.23
- net at R26.2, U2.21 (I10): now also J2.17; no longer J2.21
- net at R27.2, U2.22 (I9): now also J2.10; no longer J2.19
- net at R28.2, U2.23 (I8): now also J2.9; no longer J2.17
- net at R30.2, U2.3 (I6): now also J2.7; no longer J2.13
- net at R31.2, U2.4 (I5): now also J2.6; no longer J2.11
- net at R32.2, U2.5 (I4): now also J2.5; no longer J2.9
- net at R33.2, U2.6 (I3): now also J2.4; no longer J2.7
- net at R34.2, U2.7 (I2): now also J2.3; no longer J2.5
- net at R35.2, U2.8 (I1): now also J2.2; no longer J2.3
- net at R2.2, U8.21 (I10): now also J13.17; no longer J13.21
- net at R22.2, U1.7 (I2): now also J1.3; no longer J1.5
- net at R86.2: now also U17.6 (I3), J6.4; no longer U17.23 (I8)
- net at R94.2: now also U18.2 (I7), J9.8; no longer U18.5 (I4)
- net at R41.2, U3.2 (I7): now also J3.8; no longer J3.15
- net at R55.2, U4.4 (I5): now also J4.6; no longer J4.11
- net at R89.2: now also U17.9 (I0), J6.1; no longer U17.20 (I11)
- net at R18.2, U1.3 (I6): now also J1.7; no longer J1.13
- net at U19.21 (I10): now also R103.2, J10.17; no longer R112.2
- net at R97.2: now also U18.5 (I4), J9.5; no longer U18.2 (I7)
- net at U18.20 (I11): now also R90.2, J9.18; no longer R101.2
- net at U18.21 (I10): now also R91.2, J9.17; no longer R100.2
- net at U18.22 (I9): now also R92.2, J9.10; no longer R99.2
- net at U18.23 (I8): now also R93.2, J9.9; no longer R98.2
- net at U18.3 (I6): now also R95.2, J9.7; no longer R96.2
- net at U18.4 (I5): now also R96.2, J9.6; no longer R95.2
- net at U18.6 (I3): now also R98.2, J9.4; no longer R93.2
- net at U18.7 (I2): now also R99.2, J9.3; no longer R92.2
- net at U18.8 (I1): now also R100.2, J9.2; no longer R91.2
- net at U18.9 (I0): now also R101.2, J9.1; no longer R90.2
- net at R54.2, U4.3 (I6): now also J4.7; no longer J4.13
- net at R43.2, U3.4 (I5): now also J3.6; no longer J3.11
- net at R42.2, U3.3 (I6): now also J3.7; no longer J3.13
- net at R40.2, U3.23 (I8): now also J3.9; no longer J3.17
- net at R39.2, U3.22 (I9): now also J3.10; no longer J3.19
- net at R38.2, U3.21 (I10): now also J3.17; no longer J3.21
- net at R37.2, U3.20 (I11): now also J3.18; no longer J3.23
- net at R46.2, U3.7 (I2): now also J3.3; no longer J3.5
- net at R45.2, U3.6 (I3): now also J3.4; no longer J3.7
- net at R44.2, U3.5 (I4): now also J3.5; no longer J3.9
- net at R53.2, U4.2 (I7): now also J4.8; no longer J4.15
- net at R49.2, U4.20 (I11): now also J4.18; no longer J4.23
- net at R50.2, U4.21 (I10): now also J4.17; no longer J4.21
- net at R51.2, U4.22 (I9): now also J4.10; no longer J4.19
- net at R52.2, U4.23 (I8): now also J4.9; no longer J4.17
- net at R56.2, U4.5 (I4): now also J4.5; no longer J4.9
- net at R57.2, U4.6 (I3): now also J4.4; no longer J4.7
- net at R58.2, U4.7 (I2): now also J4.3; no longer J4.5
- net at R59.2, U4.8 (I1): now also J4.2; no longer J4.3
- net at R16.2, U1.23 (I8): now also J1.9; no longer J1.17
- net at R17.2, U1.2 (I7): now also J1.8; no longer J1.15
- net at R13.2, U1.20 (I11): now also J1.18; no longer J1.23
- net at R14.2, U1.21 (I10): now also J1.17; no longer J1.21
- net at R15.2, U1.22 (I9): now also J1.10; no longer J1.19
- net at R19.2, U1.4 (I5): now also J1.6; no longer J1.11
- net at R20.2, U1.5 (I4): now also J1.5; no longer J1.9
- net at R21.2, U1.6 (I3): now also J1.4; no longer J1.7
- net at R23.2, U1.8 (I1): now also J1.2; no longer J1.3
- net at R74.2, U5.6 (I3): now also J5.4; no longer J5.7
- net at R69.2, U5.23 (I8): now also J5.9; no longer J5.17
- net at R80.2: now also U17.22 (I9), J6.10; no longer U17.7 (I2)
- net at R110.2: now also U19.6 (I3), J10.4; no longer U19.23 (I8)
- net at R79.2: now also U17.21 (I10), J6.17; no longer U17.8 (I1)
- net at R4.2, U8.23 (I8): now also J13.9; no longer J13.17
- net at R9.2, U8.6 (I3): now also J13.4; no longer J13.7
- net at R75.2, U5.7 (I2): now also J5.3; no longer J5.5
- net at R7.2, U8.4 (I5): now also J13.6; no longer J13.11
- net at R3.2, U8.22 (I9): now also J13.10; no longer J13.19
- net at R106.2: now also U19.2 (I7), J10.8; no longer U19.5 (I4)
- net at R81.2: now also U17.23 (I8), J6.9; no longer U17.6 (I3)
- net at R78.2: now also U17.20 (I11), J6.18; no longer U17.9 (I0)
- net at R83.2: now also U17.3 (I6), J6.7; no longer U17.4 (I5)
- net at R84.2: now also U17.4 (I5), J6.6; no longer U17.3 (I6)
- net at R85.2: now also U17.5 (I4), J6.5; no longer U17.2 (I7)
- net at R87.2: now also U17.7 (I2), J6.3; no longer U17.22 (I9)
- net at R88.2: now also U17.8 (I1), J6.2; no longer U17.21 (I10)
- net at R82.2: now also U17.2 (I7), J6.8; no longer U17.5 (I4)
- net at R109.2: now also U19.5 (I4), J10.5; no longer U19.2 (I7)
- net at R113.2: now also U19.9 (I0), J10.1; no longer U19.20 (I11)
- net at R111.2: now also U19.7 (I2), J10.3; no longer U19.22 (I9)
- net at U19.3 (I6): now also R107.2, J10.7; no longer R108.2
- net at U19.4 (I5): now also R108.2, J10.6; no longer R107.2
- net at R105.2: now also U19.23 (I8), J10.9; no longer U19.6 (I3)
- net at R104.2: now also U19.22 (I9), J10.10; no longer U19.7 (I2)
- net at U19.8 (I1): now also R112.2, J10.2; no longer R103.2
- net at R102.2: now also U19.20 (I11), J10.18; no longer U19.9 (I0)
- net at R73.2, U5.5 (I4): now also J5.5; no longer J5.9
- net at R68.2, U5.22 (I9): now also J5.10; no longer J5.19
- net at R66.2, U5.20 (I11): now also J5.18; no longer J5.23
- net at R11.2, U8.8 (I1): now also J13.2; no longer J13.3
- net at R5.2, U8.2 (I7): now also J13.8; no longer J13.15
- net at R71.2, U5.3 (I6): now also J5.7; no longer J5.13
- net at R6.2, U8.3 (I6): now also J13.7; no longer J13.13
- net at R1.2, U8.20 (I11): now also J13.18; no longer J13.23
- net at R10.2, U8.7 (I2): now also J13.3; no longer J13.5
- net at R8.2, U8.5 (I4): now also J13.5; no longer J13.9
- net at R67.2, U5.21 (I10): now also J5.17; no longer J5.21
- net at R70.2, U5.2 (I7): now also J5.8; no longer J5.15
- net at R72.2, U5.4 (I5): now also J5.6; no longer J5.11
- net at R76.2, U5.8 (I1): now also J5.2; no longer J5.3
