File: Schematics/KiCad/Temp_sense_Project 2.0.kicad_pcb (KiCad board)
At the start: 4 copper layers, 238.1 x 109.5 mm, 189 parts, among them J1 348250240, J10 348250240, J11 348250240, J12 B5B-EH-A(LF)(SN), J2 348250240, J3 348250240, J4 348250240, J5 348250240, J6 B16B-PHDSS(LF)(SN), J8 348250240, J9 348250240, SW1 2-1977223-2, U1 CD74HC4067SM96, U10 STM32F446RET6, U11 CD74HC4067SM96, U12 CD74HC4067SM96, U13 CD74HC4067SM96, U14 CD74HC4067SM96, U15 CD74HC4067SM96, U16 LD1117S33CTR, U2 CD74HC4067SM96, U3 CD74HC4067SM96, U4 CD74HC4067SM96, U5 CD74HC4067SM96, U6 TIM 3.5-0911SM, U7 TCAN330GDCNR, U9 ISO7842FDWW, Y1 2

Commit message: Condense layout to 2 layers
Parts:
- removed ? (x4): , 
- removed ?: 348250240, 348250240:CONN_SD-34825-001_24_MOL
- removed D1: APHCM2012SYCK-F01, Vault:FP-APHCM2012SYCK-F01-MFG
- removed D2: APHD1608LZGCK, Vault:FP-APHD1608LZGCK-MFG
- removed FB1: BLM03BB750SZ1D, Vault:FP-BLM03-0_03-d0_3-IPC_C
- removed J12: B5B-EH-A(LF)(SN), Vault:FP-B5B-EH-A_LF_SN-MFG
- removed SW1: 2-1977223-2, Vault:FP-2-1977223-2-MFG
- removed U13, U14, U15: CD74HC4067SM96, Vault:FP-DB0024A-IPC_C
- removed U16: LD1117S33CTR, Vault:FP-SOT-223-0046067_14-MFG
- removed U6: TIM 3.5-0911SM, Vault:TIM 3.5SM SINGLE_TRP
- removed U9: ISO7842FDWW, Vault:FP-DWW0016A-MFG
- removed Y1: 2, Vault:FP-ABLS-MFG
- added C27: 2.2u, Capacitor_SMD:C_0603_1608Metric, F.Cu at (202.4, 107.8)
- added C28: 0.1u, Capacitor_SMD:C_0603_1608Metric, F.Cu at (228.9, 72.8)
- added C29: 0.1u, Capacitor_SMD:C_0603_1608Metric, F.Cu at (250.4, 70.8)
- added D3: LED, LED_SMD:LED_0603_1608Metric, F.Cu at (205.3, 105.8)
- added D4: LED, LED_SMD:LED_0603_1608Metric, F.Cu at (206.8, 104.3)
- added F2: 3A, Fuse:Fuse_0603_1608Metric, F.Cu at (258.4, 76.3)
- added FB2: 75, Resistor_SMD:R_0603_1608Metric, F.Cu at (186.4, 96.3)
- added H1: MountingHole, MountingHole:MountingHole_6.4mm_M6, F.Cu at (216.9, 57.3)
- added H2: MountingHole, MountingHole:MountingHole_6.4mm_M6, F.Cu at (53.4, 57.3)
- added H3: MountingHole, MountingHole:MountingHole_6.4mm_M6, F.Cu at (53.4, 143.3)
- added H4: MountingHole, MountingHole:MountingHole_6.4mm_M6, F.Cu at (205.4, 116.8)
- added J13: 348260240, TempSenseFootprints:CONN_SD-34826-001_24_MOL, F.Cu at (204.6, 65.5)
- added J7: Conn_02x08_Odd_Even, Connector_PinSocket_2.00mm:PinSocket_2x08_P2.00mm_Vertical, F.Cu at (260.9, 68.3)
- added Q1: 2N7002H, Package_TO_SOT_SMD:SOT-23, F.Cu at (253.8, 76.4)
- added Q2: 2N7002H, Package_TO_SOT_SMD:SOT-23, F.Cu at (253.8, 72.4)
- added R125: 3k, Resistor_SMD:R_0603_1608Metric, F.Cu at (65.9, 104.3)
- added R126: 4.7k, Resistor_SMD:R_0603_1608Metric, F.Cu at (228.4, 78.8)
- added R127: 10k, Resistor_SMD:R_0603_1608Metric, F.Cu at (250.4, 76.3)
- added R128: 120, Resistor_SMD:R_0603_1608Metric, F.Cu at (257.4, 72.3)
- added U17: CD74HC4067SM, Package_SO:SSOP-24_5.3x8.2mm_P0.65mm, F.Cu at (157.9, 122.8)
- added U18: CD74HC4067SM, Package_SO:SSOP-24_5.3x8.2mm_P0.65mm, F.Cu at (122.4, 122.8)
- added U19: CD74HC4067SM, Package_SO:SSOP-24_5.3x8.2mm_P0.65mm, F.Cu at (85.4, 122.8)
- added U20: CD74HC4067SM, Package_SO:SSOP-24_5.3x8.2mm_P0.65mm, F.Cu at (76.1, 115.5)
- added U8: CD74HC4067SM, Package_SO:SSOP-24_5.3x8.2mm_P0.65mm, F.Cu at (192.4, 78.3)
- C1: value 1210ZC106KAT2A -> 10u; footprint Vault:FP-1210-L_3_3_0_4-W_2_5_0-IPC_A -> Capacitor_SMD:C_0603_1608Metric; moved to B.Cu
- C10, C11, C8, C9: value GRM033R61A104KE15D -> 10u; footprint Vault:FP-GRM033-0_03-IPC_C -> Capacitor_SMD:C_0603_1608Metric
- C12, C14, C18, C3, C4, C5, C6, C7: value GRM033R61A104KE15D -> 100n; footprint Vault:FP-GRM033-0_03-IPC_C -> Capacitor_SMD:C_0603_1608Metric
- C13, C2: value 06035A300JAT2A -> 100n; footprint Vault:CAPC1608X90X35LL15T15 -> Capacitor_SMD:C_0603_1608Metric
- C15: value 0805YD105MAT2A -> 100n; footprint Vault:CAPC2013X140X50NL20T25 -> Capacitor_SMD:C_0603_1608Metric
- C16: value GRM033R61A104KE15D -> 1u; footprint Vault:FP-GRM033-0_03-IPC_C -> Capacitor_SMD:C_0603_1608Metric
- C17: value CC0603KPX5R7BB225 -> 100n; footprint Vault:FP-CC0603-DA-MFG -> Capacitor_SMD:C_0603_1608Metric
- C19, C20, C22, C23, C24: value 1210ZC106KAT2A -> 100n; footprint Vault:FP-1210-L_3_3_0_4-W_2_5_0-IPC_A -> Capacitor_SMD:C_0603_1608Metric
- C21: value RM033R61A104KE15D -> 1u; footprint Vault:FP-GRM033-0_03-IPC_C -> Capacitor_SMD:C_0603_1608Metric
- C25, C26: value GRM033R61A104KE15D -> 30pF; footprint Vault:FP-GRM033-0_03-IPC_C -> Capacitor_SMD:C_0603_1608Metric
- F1: value 1206L075/16WR -> 3557-2; footprint Vault:FP-1206L-MFG -> Personal:FUSE_3557-2
- J1, J10, J11, J2, J3, J4, J5, J9: value 348250240 -> 348260240; footprint 348250240:CONN_SD-34825-001_24_MOL -> TempSenseFootprints:CONN_SD-34826-001_24_MOL
- J6: value B16B-PHDSS(LF)(SN) -> 348260240; footprint Vault:FP-B16B-PHDSS_LF_SN-MFG -> TempSenseFootprints:CONN_SD-34826-001_24_MOL
- J8: value 348250240 -> Conn_01x04_Pin; footprint 348250240:CONN_SD-34825-001_24_MOL -> Connector_PinHeader_2.54mm:PinHeader_1x04_P2.54mm_Vertical
- PS1: footprint R-78E3.3-0.5:CONV_R-78E3.3-0.5 -> Converter_DCDC:Converter_DCDC_RECOM_R-78E-0.5_THT
- PS2: value R-78E3.3-0.5 -> KWS-1205-3k; footprint R-78E3.3-0.5:CONV_R-78E3.3-0.5 -> TempSenseFootprints:KWS-1205-3K
- R1, R10, R100, R101, R102, R103, R104, R105, R106, R107, R108, R109, R11, R110, R111, R112, R113, R114, R115, R116, R117, R118, R119, R12, R120, R13, R14, R15, R16, R17, R18, R19, R2, R20, R21, R22, R23, R24, R25, R26, R27, R28, R29, R3, R30, R31, R32, R33, R34, R35, R36, R37, R38, R39, R4, R40, R41, R42, R43, R44, R45, R46, R47, R48, R49, R5, R50, R51, R52, R53, R54, R55, R56, R57, R58, R59, R6, R60, R66, R67, R68, R69, R7, R70, R71, R72, R73, R74, R75, R76, R77, R78, R79, R8, R80, R81, R82, R83, R84, R85, R86, R87, R88, R89, R9, R90, R91, R92, R93, R94, R95, R96, R97, R98, R99: value RN73R2BTTD3001B25 -> 3k; footprint Vault:FP-RN73R2B-IPC_A -> Resistor_SMD:R_0603_1608Metric
- R121: value RQ73C1J100KBTD -> 3k; footprint Vault:FP-RQ731J-IPC_C -> Resistor_SMD:R_0603_1608Metric
- R122, R123: value ERJH3GJ331V -> 3k; footprint Vault:FP-ERJH3G-MFG -> Resistor_SMD:R_0603_1608Metric
- R124: value RN73C1J10KB -> 3k; footprint Vault:FP-RN731J-MFG -> Resistor_SMD:R_0603_1608Metric
- R61: value RN73R2BTTD3001B25 -> 10k; footprint Vault:FP-RN73R2B-IPC_A -> Resistor_SMD:R_0603_1608Metric
- R62, R63: value RN73R2BTTD3001B25 -> 330; footprint Vault:FP-RN73R2B-IPC_A -> Resistor_SMD:R_0603_1608Metric
- R64: value RN73R2BTTD3001B25 -> 100k; footprint Vault:FP-RN73R2B-IPC_A -> Resistor_SMD:R_0603_1608Metric
- R65: value RN73R2BTTD3001B25 -> 4.7k; footprint Vault:FP-RN73R2B-IPC_A -> Resistor_SMD:R_0603_1608Metric
- U1, U2, U3, U4, U5: value CD74HC4067SM96 -> CD74HC4067SM; footprint Vault:FP-DB0024A-IPC_C -> Package_SO:SSOP-24_5.3x8.2mm_P0.65mm
- U10: value STM32F446RET6 -> TCAN330G; footprint Vault:STM-LQFP64_L -> Package_SO:JEITA_SOIC-8_3.9x4.9mm_P1.27mm
- U11: value CD74HC4067SM96 -> STM32F446RETx; footprint Vault:FP-DB0024A-IPC_C -> Package_QFP:LQFP-64_10x10mm_P0.5mm
- U12: value CD74HC4067SM96 -> LD1117S33TR_SOT223; footprint Vault:FP-DB0024A-IPC_C -> Package_TO_SOT_SMD:SOT-223-3_TabPin2
- U7: value TCAN330GDCNR -> ISO7841FDWW; footprint Vault:FP-DCN0008A-MFG -> TempSenseFootprints:DWW0016A_N
- moved R124 183.9 mm to (65.9, 106.9), turned to 180 degrees
- moved R12 176.4 mm to (206.3, 68.8)
- moved R11 171.2 mm to (203.7, 68.8)
- moved R49 168.2 mm to (65.9, 83.9), turned to 180 degrees
- moved R50 166.1 mm to (65.9, 81.3), turned to 180 degrees
- moved R10 166.0 mm to (201.0, 68.8)
- moved R9 160.9 mm to (198.3, 68.8)
- moved R51 159.1 mm to (65.9, 97.1), turned to 180 degrees
- moved R52 156.9 mm to (65.9, 94.5), turned to 180 degrees
- moved R8 155.7 mm to (195.6, 68.8)
- moved R53 154.7 mm to (65.9, 91.8), turned to 180 degrees
- moved R54 152.5 mm to (65.9, 89.2), turned to 180 degrees
- moved R55 150.4 mm to (65.9, 86.6), turned to 180 degrees
- moved R56 150.1 mm to (65.9, 78.6), turned to 180 degrees
- moved C12 149.7 mm to (198.9, 89.8), turned to 45 degrees
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Connections:
- C1 pad 1: NetC1_1 -> +12V
- C1 pad 2: LV_GND -> GNDPWR
- C10 pad 1: NetC10_1 -> +3.3VP
- C11 pad 1: NetC11_1 -> +3V3
- C12 pad 1: NetC12_1 -> +3V3
- C13 pad 1: GND -> /MCU/MUX 3
- C13 pad 2: NetC13_2 -> GND
- C14 pad 1: NetC14_1 -> /MCU/NRST
- C15 pad 1: GND -> +3.3VA
- C15 pad 2: NetC15_2 -> GND
- C16 pad 1: NetC15_2 -> +3.3VA
- C17 pad 1: NetC17_1 -> /MCU/MUX 2
- C18 pad 1: NetC18_1 -> +3V3
- C19 pad 1: GND -> +3V3
- C19 pad 2: NetC19_2 -> GND
- C2 pad 1: NetC2_1 -> /MCU/MUX 5
- C20 pad 1: NetC20_1 -> +3V3
- C21 pad 1: NetC18_1 -> +3V3
- C22 pad 1: GND -> /MCU/MUX 1
- C22 pad 2: NetC19_2 -> GND
- C23 pad 1: NetC1_1 -> +3V3
- C23 pad 2: LV_GND -> GND
- C24 pad 1: NetC24_1 -> /MCU/MUX 0
- C24 pad 2: LV_GND -> GND
- C25 pad 1: NetC18_1 -> Net-(U11-PH0)
- C26 pad 1: NetC18_1 -> Net-(U11-PH1)
- C3 pad 1: NetC3_1 -> /MCU/MUX 6
- C4 pad 1: NetC4_1 -> /MCU/MUX 7
- C5 pad 1: NetC5_1 -> /MCU/MUX 8
- C6 pad 1: NetC6_1 -> /MCU/MUX 9
- C7 pad 1: NetC7_1 -> /MCU/MUX 4
- C8 pad 1: NetC8_1 -> +5V
- C9 pad 1: NetC9_1 -> +12V
- C9 pad 2: GND -> GNDPWR
- J1 pad 1: NetJ1_1 -> Net-(U1-I0)
- J1 pad 10: GND -> Net-(U1-I9)
- J1 pad 11: NetJ1_11 -> GND
- J1 pad 13: NetJ1_13 -> GND
- J1 pad 15: NetJ1_15 -> GND
- J1 pad 17: NetJ1_17 -> Net-(U1-I10)
- J1 pad 18: GND -> Net-(U1-I11)
- J1 pad 19: NetJ1_19 -> GND
- J1 pad 2: GND -> Net-(U1-I1)
- J1 pad 21: NetJ1_21 -> GND
- J1 pad 23: NetJ1_23 -> GND
- J1 pad 3: NetJ1_3 -> Net-(U1-I2)
- J1 pad 4: GND -> Net-(U1-I3)
- J1 pad 5: NetJ1_5 -> Net-(U1-I4)
- J1 pad 6: GND -> Net-(U1-I5)
- J1 pad 7: NetJ1_7 -> Net-(U1-I6)
- J1 pad 8: GND -> Net-(U1-I7)
- J1 pad 9: NetJ1_9 -> Net-(U1-I8)
- J10 pad 1: NetJ10_1 -> Net-(U19-I0)
- J10 pad 10: GND -> Net-(U19-I9)
- J10 pad 11: NetJ10_11 -> GND
- J10 pad 13: NetJ10_13 -> GND
- J10 pad 15: NetJ10_15 -> GND
- J10 pad 17: NetJ10_17 -> Net-(U19-I10)
- J10 pad 18: GND -> Net-(U19-I11)
- J10 pad 19: NetJ10_19 -> GND
- J10 pad 2: GND -> Net-(U19-I1)
- J10 pad 21: NetJ10_21 -> GND
- J10 pad 23: NetJ10_23 -> GND
- J10 pad 3: NetJ10_3 -> Net-(U19-I2)
- J10 pad 4: GND -> Net-(U19-I3)
- J10 pad 5: NetJ10_5 -> Net-(U19-I4)
- J10 pad 6: GND -> Net-(U19-I5)
- J10 pad 7: NetJ10_7 -> Net-(U19-I6)
- J10 pad 8: GND -> Net-(U19-I7)
- J10 pad 9: NetJ10_9 -> Net-(U19-I8)
- J11 pad 1: NetJ11_1 -> Net-(U20-I0)
- J11 pad 10: GND -> Net-(U20-I9)
- J11 pad 11: NetJ11_11 -> GND
- J11 pad 13: NetJ11_13 -> GND
- J11 pad 15: NetJ11_15 -> GND
- J11 pad 17: NetJ11_17 -> Net-(U20-I10)
- J11 pad 18: GND -> Net-(U20-I11)
- J11 pad 19: NetJ11_19 -> GND
- J11 pad 2: GND -> Net-(U20-I1)
- J11 pad 21: NetJ11_21 -> GND
- J11 pad 23: NetJ11_23 -> GND
- J11 pad 3: NetJ11_3 -> Net-(U20-I2)
- J11 pad 4: GND -> Net-(U20-I3)
- J11 pad 5: NetJ11_5 -> Net-(U20-I4)
- J11 pad 6: GND -> Net-(U20-I5)
- J11 pad 7: NetJ11_7 -> Net-(U20-I6)
- J11 pad 8: GND -> Net-(U20-I7)
- J11 pad 9: NetJ11_9 -> Net-(U20-I8)
- J2 pad 1: NetJ2_1 -> Net-(U2-I0)
- J2 pad 10: GND -> Net-(U2-I9)
- J2 pad 11: NetJ2_11 -> GND
- J2 pad 13: NetJ2_13 -> GND
- J2 pad 15: NetJ2_15 -> GND
- J2 pad 17: NetJ2_17 -> Net-(U2-I10)
- J2 pad 18: GND -> Net-(U2-I11)
- J2 pad 19: NetJ2_19 -> GND
- J2 pad 2: GND -> Net-(U2-I1)
- J2 pad 21: NetJ2_21 -> GND
- J2 pad 23: NetJ2_23 -> GND
- J2 pad 3: NetJ2_3 -> Net-(U2-I2)
- J2 pad 4: GND -> Net-(U2-I3)
- J2 pad 5: NetJ2_5 -> Net-(U2-I4)
- J2 pad 6: GND -> Net-(U2-I5)
- J2 pad 7: NetJ2_7 -> Net-(U2-I6)
- J2 pad 8: GND -> Net-(U2-I7)
- J2 pad 9: NetJ2_9 -> Net-(U2-I8)
- J3 pad 1: NetJ3_1 -> Net-(U3-I0)
- J3 pad 10: GND -> Net-(U3-I9)
- J3 pad 11: NetJ3_11 -> GND
- J3 pad 13: NetJ3_13 -> GND
- J3 pad 15: NetJ3_15 -> GND
- J3 pad 17: NetJ3_17 -> Net-(U3-I10)
- J3 pad 18: GND -> Net-(U3-I11)
- J3 pad 19: NetJ3_19 -> GND
- J3 pad 2: GND -> Net-(U3-I1)
- J3 pad 21: NetJ3_21 -> GND
- J3 pad 23: NetJ3_23 -> GND
- J3 pad 3: NetJ3_3 -> Net-(U3-I2)
- J3 pad 4: GND -> Net-(U3-I3)
- J3 pad 5: NetJ3_5 -> Net-(U3-I4)
- J3 pad 6: GND -> Net-(U3-I5)
- J3 pad 7: NetJ3_7 -> Net-(U3-I6)
- J3 pad 8: GND -> Net-(U3-I7)
- J3 pad 9: NetJ3_9 -> Net-(U3-I8)
- J4 pad 1: NetJ4_1 -> Net-(U4-I0)
- J4 pad 10: GND -> Net-(U4-I9)
- J4 pad 11: NetJ4_11 -> GND
- J4 pad 13: NetJ4_13 -> GND
- J4 pad 15: NetJ4_15 -> GND
- J4 pad 17: NetJ4_17 -> Net-(U4-I10)
- J4 pad 18: GND -> Net-(U4-I11)
- J4 pad 19: NetJ4_19 -> GND
- J4 pad 2: GND -> Net-(U4-I1)
- J4 pad 21: NetJ4_21 -> GND
- J4 pad 23: NetJ4_23 -> GND
- J4 pad 3: NetJ4_3 -> Net-(U4-I2)
- J4 pad 4: GND -> Net-(U4-I3)
- J4 pad 5: NetJ4_5 -> Net-(U4-I4)
- J4 pad 6: GND -> Net-(U4-I5)
- J4 pad 7: NetJ4_7 -> Net-(U4-I6)
- J4 pad 8: GND -> Net-(U4-I7)
- J4 pad 9: NetJ4_9 -> Net-(U4-I8)
- J5 pad 1: NetJ5_1 -> Net-(U5-I0)
- J5 pad 10: GND -> Net-(U5-I9)
- J5 pad 11: NetJ5_11 -> GND
- J5 pad 13: NetJ5_13 -> GND
- J5 pad 15: NetJ5_15 -> GND
- J5 pad 17: NetJ5_17 -> Net-(U5-I10)
- J5 pad 18: GND -> Net-(U5-I11)
- J5 pad 19: NetJ5_19 -> GND
- J5 pad 2: GND -> Net-(U5-I1)
- J5 pad 21: NetJ5_21 -> GND
- J5 pad 23: NetJ5_23 -> GND
- J5 pad 3: NetJ5_3 -> Net-(U5-I2)
- J5 pad 4: GND -> Net-(U5-I3)
- J5 pad 5: NetJ5_5 -> Net-(U5-I4)
- J5 pad 6: GND -> Net-(U5-I5)
- J5 pad 7: NetJ5_7 -> Net-(U5-I6)
- J5 pad 8: GND -> Net-(U5-I7)
- J5 pad 9: NetJ5_9 -> Net-(U5-I8)
- J6 pad 1: NetF1_1 -> Net-(U17-I0)
- J6 pad 10: (no net) -> Net-(U17-I9)
- J6 pad 11: (no net) -> GND
- J6 pad 12: (no net) -> GND
- J6 pad 13: LV_GND -> GND
- J6 pad 14: (no net) -> GND
- J6 pad 15: (no net) -> GND
- J6 pad 16: (no net) -> GND
- J6 pad 2: (no net) -> Net-(U17-I1)
- J6 pad 3: (no net) -> Net-(U17-I2)
- J6 pad 4: (no net) -> Net-(U17-I3)
- J6 pad 5: (no net) -> Net-(U17-I4)
- J6 pad 6: (no net) -> Net-(U17-I5)
- J6 pad 7: NetJ6_7 -> Net-(U17-I6)
- J6 pad 8: (no net) -> Net-(U17-I7)
- J6 pad 9: NetJ6_9 -> Net-(U17-I8)
- J8 pad 1: NetJ8_1 -> GND
- J8 pad 2: GND -> /MCU/SWCLK
- J8 pad 3: NetJ8_3 -> /MCU/SWDIO
- J8 pad 4: GND -> +5V
- J9 pad 1: NetJ9_1 -> Net-(U18-I0)
- J9 pad 10: GND -> Net-(U18-I9)
- J9 pad 11: NetJ9_11 -> GND
- J9 pad 13: NetJ9_13 -> GND
- J9 pad 15: NetJ9_15 -> GND
- J9 pad 17: NetJ9_17 -> Net-(U18-I10)
- J9 pad 18: GND -> Net-(U18-I11)
- J9 pad 19: NetJ9_19 -> GND
- J9 pad 2: GND -> Net-(U18-I1)
- J9 pad 21: NetJ9_21 -> GND
- J9 pad 23: NetJ9_23 -> GND
- J9 pad 3: NetJ9_3 -> Net-(U18-I2)
- J9 pad 4: GND -> Net-(U18-I3)
- J9 pad 5: NetJ9_5 -> Net-(U18-I4)
- J9 pad 6: GND -> Net-(U18-I5)
- J9 pad 7: NetJ9_7 -> Net-(U18-I6)
- J9 pad 8: GND -> Net-(U18-I7)
- J9 pad 9: NetJ9_9 -> Net-(U18-I8)
- PS1 pad 1: NetC1_1 -> +12V
- PS1 pad 2: LV_GND -> GNDPWR
- PS1 pad 3: NetC24_1 -> +3.3VP
- PS2 pad 1: NetC19_2 -> +12V
- PS2 pad 2: GND -> GNDPWR
- PS2 pad 3: NetC20_1 -> +5V
- R1 pad 1: NetC20_1 -> +3V3
- R1 pad 2: NetJ1_1 -> Net-(U8-I11)
- R10 pad 1: NetC20_1 -> +3V3
- R10 pad 2: NetJ1_19 -> Net-(U8-I2)
- R100 pad 1: NetC20_1 -> +3V3
- R100 pad 2: NetJ10_7 -> Net-(U18-I1)
- R101 pad 1: NetC20_1 -> +3V3
- R101 pad 2: NetJ10_9 -> Net-(U18-I0)
- R102 pad 1: NetC20_1 -> +3V3
- R102 pad 2: NetJ10_11 -> Net-(U19-I11)
- R103 pad 1: NetC20_1 -> +3V3
- R103 pad 2: NetJ10_13 -> Net-(U19-I10)
- R104 pad 1: NetC20_1 -> +3V3
- R104 pad 2: NetJ10_15 -> Net-(U19-I9)
- R105 pad 1: NetC20_1 -> +3V3
- R105 pad 2: NetJ10_17 -> Net-(U19-I8)
- R106 pad 1: NetC20_1 -> +3V3
- R106 pad 2: NetJ10_19 -> Net-(U19-I7)
- R107 pad 1: NetC20_1 -> +3V3
- R107 pad 2: NetJ10_21 -> Net-(U19-I6)
- R108 pad 1: NetC20_1 -> +3V3
- R108 pad 2: NetJ10_23 -> Net-(U19-I5)
- R109 pad 1: NetC20_1 -> +3V3
- R109 pad 2: NetJ11_1 -> Net-(U19-I4)
- R11 pad 1: NetC20_1 -> +3V3
- R11 pad 2: NetJ1_21 -> Net-(U8-I1)
- R110 pad 1: NetC20_1 -> +3V3
- R110 pad 2: NetJ11_3 -> Net-(U19-I3)
- R111 pad 1: NetC20_1 -> +3V3
- R111 pad 2: NetJ11_5 -> Net-(U19-I2)
- R112 pad 1: NetC20_1 -> +3V3
- R112 pad 2: NetJ11_7 -> Net-(U19-I1)
- R113 pad 1: NetC20_1 -> +3V3
- R113 pad 2: NetJ11_9 -> Net-(U19-I0)
- R114 pad 1: NetC20_1 -> +3V3
- R114 pad 2: NetJ11_11 -> Net-(U20-I11)
- R115 pad 1: NetC20_1 -> +3V3
- R115 pad 2: NetJ11_13 -> Net-(U20-I10)
- R116 pad 1: NetC20_1 -> +3V3
- R116 pad 2: NetJ11_15 -> Net-(U20-I9)
- R117 pad 1: NetC20_1 -> +3V3
- R117 pad 2: NetJ11_17 -> Net-(U20-I8)
- R118 pad 1: NetC20_1 -> +3V3
- R118 pad 2: NetJ11_19 -> Net-(U20-I7)
- R119 pad 1: NetC20_1 -> +3V3
- R119 pad 2: NetJ11_21 -> Net-(U20-I6)
- R12 pad 1: NetC20_1 -> +3V3
- R12 pad 2: NetJ1_23 -> Net-(U8-I0)
- R120 pad 1: NetC20_1 -> +3V3
- R120 pad 2: NetJ11_23 -> Net-(U20-I5)
- R121 pad 1: GND -> +3V3
- R121 pad 2: NetR121_2 -> Net-(U20-I4)
- R122 pad 1: NetC18_1 -> +3V3
- R122 pad 2: NetD1_2 -> Net-(U20-I3)
- R123 pad 1: NetC18_1 -> +3V3
- R123 pad 2: NetD2_2 -> Net-(U20-I2)
- R124 pad 1: NetR124_1 -> +3V3
- R124 pad 2: NetC24_1 -> Net-(U20-I1)
- R13 pad 1: NetC20_1 -> +3V3
- R13 pad 2: NetJ2_1 -> Net-(U1-I11)
- R14 pad 1: NetC20_1 -> +3V3
- R14 pad 2: NetJ2_3 -> Net-(U1-I10)
- R15 pad 1: NetC20_1 -> +3V3
- R15 pad 2: NetJ2_5 -> Net-(U1-I9)
- R16 pad 1: NetC20_1 -> +3V3
- R16 pad 2: NetJ2_7 -> Net-(U1-I8)
- R17 pad 1: NetC20_1 -> +3V3
- R17 pad 2: NetJ2_9 -> Net-(U1-I7)
- R18 pad 1: NetC20_1 -> +3V3
- R18 pad 2: NetJ2_11 -> Net-(U1-I6)
- R19 pad 1: NetC20_1 -> +3V3
- R19 pad 2: NetJ2_13 -> Net-(U1-I5)
- R2 pad 1: NetC20_1 -> +3V3
- R2 pad 2: NetJ1_3 -> Net-(U8-I10)
- R20 pad 1: NetC20_1 -> +3V3
- R20 pad 2: NetJ2_15 -> Net-(U1-I4)
- R21 pad 1: NetC20_1 -> +3V3
- R21 pad 2: NetJ2_17 -> Net-(U1-I3)
- R22 pad 1: NetC20_1 -> +3V3
- R22 pad 2: NetJ2_19 -> Net-(U1-I2)
- R23 pad 1: NetC20_1 -> +3V3
- R23 pad 2: NetJ2_21 -> Net-(U1-I1)
- R24 pad 1: NetC20_1 -> +3V3
- R24 pad 2: NetJ2_23 -> Net-(U1-I0)
- R25 pad 1: NetC20_1 -> +3V3
- R25 pad 2: NetJ3_1 -> Net-(U2-I11)
- R26 pad 1: NetC20_1 -> +3V3
- R26 pad 2: NetJ3_3 -> Net-(U2-I10)
- R27 pad 1: NetC20_1 -> +3V3
- R27 pad 2: NetJ3_5 -> Net-(U2-I9)
- R28 pad 1: NetC20_1 -> +3V3
- R28 pad 2: NetJ3_7 -> Net-(U2-I8)
- R29 pad 1: NetC20_1 -> +3V3
- R29 pad 2: NetJ3_9 -> Net-(U2-I7)
- R3 pad 1: NetC20_1 -> +3V3
- R3 pad 2: NetJ1_5 -> Net-(U8-I9)
- R30 pad 1: NetC20_1 -> +3V3
- R30 pad 2: NetJ3_11 -> Net-(U2-I6)
- R31 pad 1: NetC20_1 -> +3V3
- R31 pad 2: NetJ3_13 -> Net-(U2-I5)
- R32 pad 1: NetC20_1 -> +3V3
- R32 pad 2: NetJ3_15 -> Net-(U2-I4)
- R33 pad 1: NetC20_1 -> +3V3
- R33 pad 2: NetJ3_17 -> Net-(U2-I3)
- R34 pad 1: NetC20_1 -> +3V3
- R34 pad 2: NetJ3_19 -> Net-(U2-I2)
- R35 pad 1: NetC20_1 -> +3V3
- R35 pad 2: NetJ3_21 -> Net-(U2-I1)
- R36 pad 1: NetC20_1 -> +3V3
- R36 pad 2: NetJ3_23 -> Net-(U2-I0)
- R37 pad 1: NetC20_1 -> +3V3
- R37 pad 2: NetJ4_1 -> Net-(U3-I11)
- R38 pad 1: NetC20_1 -> +3V3
- R38 pad 2: NetJ4_3 -> Net-(U3-I10)
- R39 pad 1: NetC20_1 -> +3V3
- R39 pad 2: NetJ4_5 -> Net-(U3-I9)
- R4 pad 1: NetC20_1 -> +3V3
- R4 pad 2: NetJ1_7 -> Net-(U8-I8)
- R40 pad 1: NetC20_1 -> +3V3
- R40 pad 2: NetJ4_7 -> Net-(U3-I8)
- R41 pad 1: NetC20_1 -> +3V3
- R41 pad 2: NetJ4_9 -> Net-(U3-I7)
- R42 pad 1: NetC20_1 -> +3V3
- R42 pad 2: NetJ4_11 -> Net-(U3-I6)
- R43 pad 1: NetC20_1 -> +3V3
- R43 pad 2: NetJ4_13 -> Net-(U3-I5)
- R44 pad 1: NetC20_1 -> +3V3
- R44 pad 2: NetJ4_15 -> Net-(U3-I4)
- R45 pad 1: NetC20_1 -> +3V3
- R45 pad 2: NetJ4_17 -> Net-(U3-I3)
- R46 pad 1: NetC20_1 -> +3V3
- R46 pad 2: NetJ4_19 -> Net-(U3-I2)
- R47 pad 1: NetC20_1 -> +3V3
- R47 pad 2: NetJ4_21 -> Net-(U3-I1)
- R48 pad 1: NetC20_1 -> +3V3
- R48 pad 2: NetJ4_23 -> Net-(U3-I0)
- R49 pad 1: NetC20_1 -> +3V3
- R49 pad 2: NetJ5_1 -> Net-(U4-I11)
- R5 pad 1: NetC20_1 -> +3V3
- R5 pad 2: NetJ1_9 -> Net-(U8-I7)
- R50 pad 1: NetC20_1 -> +3V3
- R50 pad 2: NetJ5_3 -> Net-(U4-I10)
- R51 pad 1: NetC20_1 -> +3V3
- R51 pad 2: NetJ5_5 -> Net-(U4-I9)
- R52 pad 1: NetC20_1 -> +3V3
- R52 pad 2: NetJ5_7 -> Net-(U4-I8)
- R53 pad 1: NetC20_1 -> +3V3
- R53 pad 2: NetJ5_9 -> Net-(U4-I7)
- R54 pad 1: NetC20_1 -> +3V3
- R54 pad 2: NetJ5_11 -> Net-(U4-I6)
- R55 pad 1: NetC20_1 -> +3V3
- R55 pad 2: NetJ5_13 -> Net-(U4-I5)
- R56 pad 1: NetC20_1 -> +3V3
- R56 pad 2: NetJ5_15 -> Net-(U4-I4)
- R57 pad 1: NetC20_1 -> +3V3
- R57 pad 2: NetJ5_17 -> Net-(U4-I3)
- R58 pad 1: NetC20_1 -> +3V3
- R58 pad 2: NetJ5_19 -> Net-(U4-I2)
- R59 pad 1: NetC20_1 -> +3V3
- R59 pad 2: NetJ5_21 -> Net-(U4-I1)
- R6 pad 1: NetC20_1 -> +3V3
- R6 pad 2: NetJ1_11 -> Net-(U8-I6)
- R60 pad 1: NetC20_1 -> +3V3
- R60 pad 2: NetJ5_23 -> Net-(U4-I0)
- R61 pad 1: NetC20_1 -> Net-(Q2-G)
- R61 pad 2: NetJ7_1 -> GNDPWR
- R62 pad 1: NetC20_1 -> +3V3
- R62 pad 2: NetJ7_3 -> Net-(D3-A)
- R63 pad 1: NetC20_1 -> +3V3
- R63 pad 2: NetJ7_5 -> Net-(D4-A)
- R64 pad 1: NetC20_1 -> /MCU/BOOT0
- R64 pad 2: NetJ7_7 -> GND
- R65 pad 1: NetC20_1 -> +3.3VP
- R65 pad 2: NetJ7_9 -> Net-(U7-EN2)
- R66 pad 1: NetC20_1 -> +3V3
- R66 pad 2: NetJ7_11 -> Net-(U5-I11)
- R67 pad 1: NetC20_1 -> +3V3
- R67 pad 2: NetJ7_13 -> Net-(U5-I10)
- R68 pad 1: NetC20_1 -> +3V3
- R68 pad 2: NetJ7_15 -> Net-(U5-I9)
- R69 pad 1: NetC20_1 -> +3V3
- R69 pad 2: NetJ7_17 -> Net-(U5-I8)
- R7 pad 1: NetC20_1 -> +3V3
- R7 pad 2: NetJ1_13 -> Net-(U8-I5)
- R70 pad 1: NetC20_1 -> +3V3
- R70 pad 2: NetJ7_19 -> Net-(U5-I7)
- R71 pad 1: NetC20_1 -> +3V3
- R71 pad 2: NetJ7_21 -> Net-(U5-I6)
- R72 pad 1: NetC20_1 -> +3V3
- R72 pad 2: NetJ7_23 -> Net-(U5-I5)
- R73 pad 1: NetC20_1 -> +3V3
- R73 pad 2: NetJ8_1 -> Net-(U5-I4)
- R74 pad 1: NetC20_1 -> +3V3
- R74 pad 2: NetJ8_3 -> Net-(U5-I3)
- R75 pad 1: NetC20_1 -> +3V3
- R75 pad 2: NetJ8_5 -> Net-(U5-I2)
- R76 pad 1: NetC20_1 -> +3V3
- R76 pad 2: NetJ8_7 -> Net-(U5-I1)
- R77 pad 1: NetC20_1 -> +3V3
- R77 pad 2: NetJ8_9 -> Net-(U5-I0)
- R78 pad 1: NetC20_1 -> +3V3
- R78 pad 2: NetJ8_11 -> Net-(U17-I11)
- R79 pad 1: NetC20_1 -> +3V3
- R79 pad 2: NetJ8_13 -> Net-(U17-I10)
- R8 pad 1: NetC20_1 -> +3V3
- R8 pad 2: NetJ1_15 -> Net-(U8-I4)
- R80 pad 1: NetC20_1 -> +3V3
- R80 pad 2: NetJ8_15 -> Net-(U17-I9)
- R81 pad 1: NetC20_1 -> +3V3
- R81 pad 2: NetJ8_17 -> Net-(U17-I8)
- R82 pad 1: NetC20_1 -> +3V3
- R82 pad 2: NetJ8_19 -> Net-(U17-I7)
- R83 pad 1: NetC20_1 -> +3V3
- R83 pad 2: NetJ8_21 -> Net-(U17-I6)
- R84 pad 1: NetC20_1 -> +3V3
- R84 pad 2: NetJ8_23 -> Net-(U17-I5)
- R85 pad 1: NetC20_1 -> +3V3
- R85 pad 2: NetJ9_1 -> Net-(U17-I4)
- R86 pad 1: NetC20_1 -> +3V3
- R86 pad 2: NetJ9_3 -> Net-(U17-I3)
- R87 pad 1: NetC20_1 -> +3V3
- R87 pad 2: NetJ9_5 -> Net-(U17-I2)
- R88 pad 1: NetC20_1 -> +3V3
- R88 pad 2: NetJ9_7 -> Net-(U17-I1)
- R89 pad 1: NetC20_1 -> +3V3
- R89 pad 2: NetJ9_9 -> Net-(U17-I0)
- R9 pad 1: NetC20_1 -> +3V3
- R9 pad 2: NetJ1_17 -> Net-(U8-I3)
- R90 pad 1: NetC20_1 -> +3V3
- R90 pad 2: NetJ9_11 -> Net-(U18-I11)
- R91 pad 1: NetC20_1 -> +3V3
- R91 pad 2: NetJ9_13 -> Net-(U18-I10)
- R92 pad 1: NetC20_1 -> +3V3
- R92 pad 2: NetJ9_15 -> Net-(U18-I9)
- R93 pad 1: NetC20_1 -> +3V3
- R93 pad 2: NetJ9_17 -> Net-(U18-I8)
- R94 pad 1: NetC20_1 -> +3V3
- R94 pad 2: NetJ9_19 -> Net-(U18-I7)
- R95 pad 1: NetC20_1 -> +3V3
- R95 pad 2: NetJ9_21 -> Net-(U18-I6)
- R96 pad 1: NetC20_1 -> +3V3
- R96 pad 2: NetJ9_23 -> Net-(U18-I5)
- R97 pad 1: NetC20_1 -> +3V3
- R97 pad 2: NetJ10_1 -> Net-(U18-I4)
- R98 pad 1: NetC20_1 -> +3V3
- R98 pad 2: NetJ10_3 -> Net-(U18-I3)
- R99 pad 1: NetC20_1 -> +3V3
- R99 pad 2: NetJ10_5 -> Net-(U18-I2)
- U1 pad 1: NetC3_1 -> /MCU/MUX 6
- U1 pad 10: NetU1_10 -> /MCU/S0
- U1 pad 11: NetU1_11 -> /MCU/S1
- U1 pad 13: NetU1_13 -> /MCU/S3
- U1 pad 14: NetU1_14 -> /MCU/S2
- U1 pad 16: (no net) -> unconnected-(U1-I15-Pad16)
- U1 pad 17: (no net) -> unconnected-(U1-I14-Pad17)
- U1 pad 18: (no net) -> unconnected-(U1-I13-Pad18)
- U1 pad 19: (no net) -> unconnected-(U1-I12-Pad19)
- U1 pad 2: NetJ1_15 -> Net-(U1-I7)
- U1 pad 20: NetJ1_23 -> Net-(U1-I11)
- U1 pad 21: NetJ1_21 -> Net-(U1-I10)
- U1 pad 22: NetJ1_19 -> Net-(U1-I9)
- U1 pad 23: NetJ1_17 -> Net-(U1-I8)
- U1 pad 24: NetC20_1 -> +3V3
- U1 pad 3: NetJ1_13 -> Net-(U1-I6)
- U1 pad 4: NetJ1_11 -> Net-(U1-I5)
- U1 pad 5: NetJ1_9 -> Net-(U1-I4)
- U1 pad 6: NetJ1_7 -> Net-(U1-I3)
- U1 pad 7: NetJ1_5 -> Net-(U1-I2)
- U1 pad 8: NetJ1_3 -> Net-(U1-I1)
- U1 pad 9: NetJ1_1 -> Net-(U1-I0)
- U10 pad 1: NetC18_1 -> Net-(U10-TXD)
- U10 pad 2: (no net) -> GNDPWR
- U10 pad 3: (no net) -> +3.3VP
- U10 pad 4: (no net) -> Net-(U10-RXD)
- U10 pad 5: NetC2_1 -> +3.3VP
- U10 pad 6: NetC13_2 -> /Power and Isolation/CANL
- U10 pad 7: NetC14_1 -> /Power and Isolation/CANH
- U10 pad 8: NetC6_1 -> GNDPWR
- U11 pad 1: NetC8_1 -> +3V3
- U11 pad 10: NetU1_10 -> /MCU/MUX 7
- U11 pad 11: NetU1_11 -> /MCU/MUX 8
- U11 pad 13: NetU1_13 -> +3.3VA
- U11 pad 14: NetU1_14 -> /MCU/MUX 9
- U11 pad 15: GND -> /MCU/S0
- U11 pad 16: (no net) -> /MCU/S1
- U11 pad 17: (no net) -> /MCU/S2
- U11 pad 18: (no net) -> GND
- U11 pad 19: (no net) -> +3V3
- U11 pad 2: NetJ7_15 -> unconnected-(U11-PC13-Pad2)
- U11 pad 20: NetJ7_23 -> /MCU/S3
- U11 pad 21: NetJ7_21 -> /MCU/MUX 4
- U11 pad 22: NetJ7_19 -> /MCU/MUX 3
- U11 pad 23: NetJ7_17 -> /MCU/MUX 2
- U11 pad 24: NetC20_1 -> /MCU/MUX 1
- U11 pad 3: NetJ7_13 -> unconnected-(U11-PC14-Pad3)
- U11 pad 4: NetJ7_11 -> unconnected-(U11-PC15-Pad4)
- U11 pad 5: NetJ7_9 -> Net-(U11-PH0)
- U11 pad 6: NetJ7_7 -> Net-(U11-PH1)
- U11 pad 7: NetJ7_5 -> /MCU/NRST
- U11 pad 8: NetJ7_3 -> /MCU/MUX 5
- U11 pad 9: NetJ7_1 -> /MCU/MUX 6
- U12 pad 1: NetC9_1 -> GND
- U12 pad 2: NetJ8_15 -> +3V3
- U12 pad 3: NetJ8_13 -> +5V
- U2 pad 1: NetC4_1 -> /MCU/MUX 7
- U2 pad 10: NetU1_10 -> /MCU/S0
- U2 pad 11: NetU1_11 -> /MCU/S1
- U2 pad 13: NetU1_13 -> /MCU/S3
- U2 pad 14: NetU1_14 -> /MCU/S2
- U2 pad 16: (no net) -> unconnected-(U2-I15-Pad16)
- U2 pad 17: (no net) -> unconnected-(U2-I14-Pad17)
- U2 pad 18: (no net) -> unconnected-(U2-I13-Pad18)
- U2 pad 19: (no net) -> unconnected-(U2-I12-Pad19)
- U2 pad 2: NetJ2_15 -> Net-(U2-I7)
- U2 pad 20: NetJ2_23 -> Net-(U2-I11)
- U2 pad 21: NetJ2_21 -> Net-(U2-I10)
- U2 pad 22: NetJ2_19 -> Net-(U2-I9)
- U2 pad 23: NetJ2_17 -> Net-(U2-I8)
- U2 pad 24: NetC20_1 -> +3V3
- U2 pad 3: NetJ2_13 -> Net-(U2-I6)
- U2 pad 4: NetJ2_11 -> Net-(U2-I5)
- U2 pad 5: NetJ2_9 -> Net-(U2-I4)
- U2 pad 6: NetJ2_7 -> Net-(U2-I3)
- U2 pad 7: NetJ2_5 -> Net-(U2-I2)
- U2 pad 8: NetJ2_3 -> Net-(U2-I1)
- U2 pad 9: NetJ2_1 -> Net-(U2-I0)
- U3 pad 1: NetC5_1 -> /MCU/MUX 8
- U3 pad 10: NetU1_10 -> /MCU/S0
- U3 pad 11: NetU1_11 -> /MCU/S1
- U3 pad 13: NetU1_13 -> /MCU/S3
- U3 pad 14: NetU1_14 -> /MCU/S2
- U3 pad 16: (no net) -> unconnected-(U3-I15-Pad16)
- U3 pad 17: (no net) -> unconnected-(U3-I14-Pad17)
- U3 pad 18: (no net) -> unconnected-(U3-I13-Pad18)
- U3 pad 19: (no net) -> unconnected-(U3-I12-Pad19)
- U3 pad 2: NetJ3_15 -> Net-(U3-I7)
- U3 pad 20: NetJ3_23 -> Net-(U3-I11)
- U3 pad 21: NetJ3_21 -> Net-(U3-I10)
- U3 pad 22: NetJ3_19 -> Net-(U3-I9)
- U3 pad 23: NetJ3_17 -> Net-(U3-I8)
- U3 pad 24: NetC20_1 -> +3V3
- U3 pad 3: NetJ3_13 -> Net-(U3-I6)
- U3 pad 4: NetJ3_11 -> Net-(U3-I5)
- U3 pad 5: NetJ3_9 -> Net-(U3-I4)
- U3 pad 6: NetJ3_7 -> Net-(U3-I3)
- U3 pad 7: NetJ3_5 -> Net-(U3-I2)
- U3 pad 8: NetJ3_3 -> Net-(U3-I1)
- U3 pad 9: NetJ3_1 -> Net-(U3-I0)
- U4 pad 1: NetC6_1 -> /MCU/MUX 9
- U4 pad 10: NetU1_10 -> /MCU/S0
- U4 pad 11: NetU1_11 -> /MCU/S1
- U4 pad 13: NetU1_13 -> /MCU/S3
- U4 pad 14: NetU1_14 -> /MCU/S2
- U4 pad 16: (no net) -> unconnected-(U4-I15-Pad16)
- U4 pad 17: (no net) -> unconnected-(U4-I14-Pad17)
- U4 pad 18: (no net) -> unconnected-(U4-I13-Pad18)
- U4 pad 19: (no net) -> unconnected-(U4-I12-Pad19)
- U4 pad 2: NetJ4_15 -> Net-(U4-I7)
- U4 pad 20: NetJ4_23 -> Net-(U4-I11)
- U4 pad 21: NetJ4_21 -> Net-(U4-I10)
- U4 pad 22: NetJ4_19 -> Net-(U4-I9)
- U4 pad 23: NetJ4_17 -> Net-(U4-I8)
- U4 pad 24: NetC20_1 -> +3V3
- U4 pad 3: NetJ4_13 -> Net-(U4-I6)
- U4 pad 4: NetJ4_11 -> Net-(U4-I5)
- U4 pad 5: NetJ4_9 -> Net-(U4-I4)
- U4 pad 6: NetJ4_7 -> Net-(U4-I3)
- U4 pad 7: NetJ4_5 -> Net-(U4-I2)
- U4 pad 8: NetJ4_3 -> Net-(U4-I1)
- U4 pad 9: NetJ4_1 -> Net-(U4-I0)
- U5 pad 1: NetC7_1 -> /MCU/MUX 0
- U5 pad 10: NetU1_10 -> /MCU/S0
- U5 pad 11: NetU1_11 -> /MCU/S1
- U5 pad 13: NetU1_13 -> /MCU/S3
- U5 pad 14: NetU1_14 -> /MCU/S2
- U5 pad 16: (no net) -> unconnected-(U5-I15-Pad16)
- U5 pad 17: (no net) -> unconnected-(U5-I14-Pad17)
- U5 pad 18: (no net) -> unconnected-(U5-I13-Pad18)
- U5 pad 19: (no net) -> unconnected-(U5-I12-Pad19)
- U5 pad 2: NetJ5_15 -> Net-(U5-I7)
- U5 pad 20: NetJ5_23 -> Net-(U5-I11)
- U5 pad 21: NetJ5_21 -> Net-(U5-I10)
- U5 pad 22: NetJ5_19 -> Net-(U5-I9)
- U5 pad 23: NetJ5_17 -> Net-(U5-I8)
- U5 pad 24: NetC20_1 -> +3V3
- U5 pad 3: NetJ5_13 -> Net-(U5-I6)
- U5 pad 4: NetJ5_11 -> Net-(U5-I5)
- U5 pad 5: NetJ5_9 -> Net-(U5-I4)
- U5 pad 6: NetJ5_7 -> Net-(U5-I3)
- U5 pad 7: NetJ5_5 -> Net-(U5-I2)
- U5 pad 8: NetJ5_3 -> Net-(U5-I1)
- U5 pad 9: NetJ5_1 -> Net-(U5-I0)
- U7 pad 1: NetU7_1 -> +3V3
- U7 pad 2: LV_GND -> GND
- U7 pad 3: NetC24_1 -> /MCU/Discharge Fault
- U7 pad 4: NetU7_4 -> /MCU/Charge Fault
- U7 pad 5: NetC24_1 -> /MCU/CAN TX
- U7 pad 6: NetJ6_9 -> /MCU/CAN RX
- U7 pad 7: NetJ6_7 -> Net-(U7-EN1)
- U7 pad 8: LV_GND -> GND
Routing:
- net /MCU/S3: track 0.00 -> 130.6 mm, vias 0 -> 2
- net /MCU/S2: track 0.00 -> 127.3 mm, vias 0 -> 2
- net /MCU/S1: track 0.00 -> 125.5 mm, vias 0 -> 3
- net /MCU/MUX 9: track 0.00 -> 124.8 mm
- net /MCU/S0: track 0.00 -> 123.6 mm, vias 0 -> 3
- net /MCU/MUX 3: track 0.00 -> 120.4 mm
- net /MCU/MUX 4: track 0.00 -> 118.8 mm
- net /MCU/MUX 8: track 0.00 -> 113.2 mm
- net /MCU/MUX 2: track 0.00 -> 83.9 mm
- net /MCU/MUX 7: track 0.00 -> 80.0 mm
- net +12V: track 0.00 -> 67.1 mm
- net +3V3: track 0.00 -> 58.4 mm
- net /MCU/Charge Fault: track 0.00 -> 52.5 mm
- net /MCU/MUX 1: track 0.00 -> 50.8 mm
- net /MCU/Discharge Fault: track 0.00 -> 44.9 mm
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- added copper zone on B.Cu, net GNDPWR
- removed copper zone on B.Cu, net LV_GND
Other:
- board size 238.1 x 109.5 mm -> 220 x 99 mm
- copper layers 4 -> 2
- rule pad_to_mask_clearance: 0.1016 -> 0
- board text removed: "90 degree header space"
- board text removed: "<-9.9mm->"
- board text removed: "High Voltage"

Commit message: More pcb layout work
Parts:
- removed C25, C26: 30pF, Capacitor_SMD:C_0603_1608Metric
- added C30: 6pF, Capacitor_SMD:C_0402_1005Metric, F.Cu at (193.4, 88.3)
- added C31: 6pF, Capacitor_SMD:C_0402_1005Metric, F.Cu at (190.4, 90.8)
- added Y2: 7B008000F01, Crystal:Crystal_SMD_3225-4Pin_3.2x2.5mm, F.Cu at (193.4, 90.8)
- moved C27 7.28 mm to (195.4, 105.8), turned to -45 degrees
- moved C14 5.32 mm to (189.4, 89.3)
- moved C16 4.12 mm to (189.4, 96.8), turned to -90 degrees
- moved C15 2.70 mm to (190.9, 96.8), turned to -90 degrees
- moved R126 2.50 mm to (228.4, 81.3), turned to -90 degrees
- moved C13 1.80 mm to (81.9, 116.3), turned to 90 degrees
- moved FB2 1.58 mm to (187.9, 96.8)
- moved C2 0.71 mm to (188.9, 84.8), turned to 90 degrees
Routing:
- net /MCU/S3: track 130.6 -> 342.9 mm, vias 2 -> 7
- net /MCU/S2: track 127.3 -> 339.2 mm, vias 2 -> 18
- net /MCU/S1: track 125.5 -> 312.9 mm, vias 3 -> 11
- net /MCU/S0: track 123.6 -> 310.7 mm, vias 3 -> 11
- net +3V3: track 58.4 -> 111.6 mm
- net GND: track 23.6 -> 69.6 mm, vias 1 -> 11
- net /MCU/NRST: track 0.00 -> 9.58 mm
- net +5V: track 21.8 -> 30.2 mm
- net Net-(U11-PH1): track 0.00 -> 6.82 mm
- net Net-(U11-PH0): track 0.00 -> 6.27 mm
- net /MCU/MUX 5: track 19.1 -> 25.1 mm
- net Net-(U4-I11): track 12.2 -> 18.1 mm
- net Net-(U4-I10): track 13.9 -> 19.5 mm
- net Net-(U1-I11): track 14.3 -> 19.2 mm
- net Net-(U8-I11): track 14.2 -> 19.0 mm
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Other:
- outline, holes or cut-outs redrawn

Commit message: Get rid of excess files
Routing:
- net +3V3: track 111.6 -> 659.5 mm, vias 0 -> 120
- net /MCU/S0: track 310.7 -> 435.6 mm, vias 11 -> 27
- net /MCU/S1: track 312.9 -> 428.7 mm, vias 11 -> 29
- net GND: track 69.6 -> 159.8 mm, vias 11 -> 40
- net /MCU/S3: track 342.9 -> 400.0 mm, vias 7 -> 11
- net /MCU/S2: track 339.2 -> 396.0 mm, vias 18 -> 29
- net GNDPWR: track 41.8 -> 53.3 mm
- net +3.3VP: track 29.8 -> 35.6 mm
- net Net-(U18-I10): track 14.4 -> 19.7 mm
- net Net-(U5-I11): track 12.6 -> 17.8 mm
- net Net-(U5-I10): track 13.9 -> 18.9 mm
- net Net-(U18-I11): track 13.3 -> 18.3 mm
- net Net-(U18-I0): track 15.9 -> 19.8 mm
- net Net-(U5-I9): track 17.4 -> 21.3 mm
- net Net-(U5-I0): track 13.4 -> 17.1 mm
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- added copper zone on F.Cu, net +3V3
Other:
- outline, holes or cut-outs redrawn
